Commit message: Add realsense links.

File: robo_description/urdf/robo_camera.urdf.xacro (robot description, xacro)
@@ -6,16 +6,19 @@
   <property name="camera_offset_y" value="0.0" />
   <property name="camera_offset_z" value="0.0" />
-  <!-- Define the camera -->
   <macro name="camera" params="parent name color *origin">
-    <joint name="${parent}_${name}_joint" type="fixed">
+    <!-- Telescoping neck joint/link -->
+    <joint name="${parent}_${name}_tele_joint" type="prismatic">
       <xacro:insert_block name="origin" />
       <parent link="${parent}_link"/>
-      <child link="${name}_link"/>
+      <child link="${name}_tele_link"/>
+      <axis xyz="0 0 1" />
+      <origin xyz="0 0 0" rpy="0 0 0"/>
+      <limit lower="0" upper="0.19" velocity="0.1" effort="1.0" />
     </joint>
-    <link name="${name}_link">
+    <link name="${name}_tele_link">
       <visual>
         <origin xyz="0 0 0" rpy="0 0 0" />
         <geometry>
-           <mesh filename="package://robo_description/meshes/camera/vis/vis_camera_03.STL" scale="${scale} ${scale} ${scale}" />
+          <box size="0.01 0.01 0.25"/>
         </geometry>
         <material name="${color}" />
@@ -24,19 +27,102 @@
         <origin xyz="0 0 0" rpy="0 0 0" />
         <geometry>
+          <box size="0.02 0.02 0.5"/>
+        </geometry>
+      </collision>
+    </link>
+    <!-- Pan joint/link -->
+    <joint name="${name}_pan_joint" type="revolute">
+      <axis xyz="0 0 1"/>
+      <origin xyz="0 0 0.135" rpy="0 0 0"/>
+      <limit effort="1000.0" lower="${pi/2}" upper="${-pi/2}" velocity="0.5"/>
+      <parent link="${name}_tele_link"/>
+      <child link="${name}_pan_link"/>
+    </joint>
+    <link name="${name}_pan_link">
+      <visual>
+        <origin rpy="0 0 0" xyz="0 0 0"/>
+        <geometry>
+          <box size="0.03 0.03 0.03"/>
+        </geometry>
+        <material name="blue"/>
+      </visual>
+      <collision>
+        <origin rpy="0 0 0" xyz="0 0 0"/>
+        <geometry>
+          <box size="0.03 0.03 0.03"/>
+        </geometry>
+      </collision>
+    </link>
+    <!-- Tilt joint/link -->
+    <joint name="${name}_tilt_joint" type="revolute">
+      <axis xyz="1 0 0"/>
+      <origin xyz="0 0.01 0" rpy="0 0 0"/>
+      <limit effort="1000.0" lower="${-pi/4}" upper="${1.2*pi/2}" velocity="0.5"/>
+      <parent link="${name}_pan_link"/>
+      <child link="${name}_tilt_link"/>
+    </joint>
+    <link name="${name}_tilt_link">
+      <visual>
+        <origin xyz="0 0.012 0" rpy="0 0 0"/>
+        <geometry>
+          <box size="0.03 0.03 0.01"/>
+        </geometry>
+        <material name="green"/>
+      </visual>
+      <collision>
+        <origin rpy="0 0 0" xyz="0 0 0"/>
+        <geometry>
+          <box size="0.03 0.03 0.01"/>
+        </geometry>
+      </collision>
+    </link>
+    <!-- Realsense joint/link -->
+    <joint name="${name}_realsense_joint" type="fixed">
+      <xacro:insert_block name="origin" />
+      <parent link="${name}_tilt_link"/>
+      <child link="realsense_link"/>
+    </joint>
+    <link name="realsense_link">
+      <visual>
+        <origin xyz="0 -0.025 -0.01" rpy="0 0 0" />
+        <geometry>
+          <mesh filename="package://robo_description/meshes/camera/vis/RealSense.STL" scale="${scale} ${scale} ${scale}" />
+        </geometry>
+        <material name="${color}" />
+      </visual>
+      <collision>
+        <origin xyz="0 0 0" rpy="0 0 0" />
+        <geometry>
+          <!--box size="0.1 0.02 0.02"/-->
           <mesh filename="package://robo_description/meshes/camera/col/col_camera_03.STL" scale="${scale} ${scale} ${scale}" />
         </geometry>
       </collision>
     </link>
-    <!-- Depth and RGB frames for tf transform trees -->
-    <!-- *Need to update values to reflect RealSense/arrangement -->
+    <!-- realsense_frame -->
+    <joint name="${name}_realsense_frame_joint" type="fixed">
+      <origin xyz="0 -0.027 0" rpy="${pi/2} ${pi} 0" />
+      <xacro:insert_block name="origin" />
+      <parent link="realsense_link"/>
+      <child link="realsense_frame"/>
+    </joint>
+    <link name="realsense_frame">
+      <visual>
+        <origin xyz="0 0 0" rpy="0 0 0" />
+        <geometry>
+          <box size="0.003 0.003 0.0005"/>
+        </geometry>
+        <material name="blue" />
+      </visual>
+    </link>
+    <!-- camera_depth_optical_frame -->
     <joint name="${name}_depth_joint" type="fixed">
-      <origin xyz="0 0.0 0.268" rpy="0 0 0" />
-      <parent link="${name}_link" />
-      <child link="${name}_depth_frame" />
+      <origin xyz="0 0 0.268" rpy="0 0 0" />
+      <parent link="realsense_frame" />
+      <child link="camera_depth_optical_frame" />
     </joint>
-    <link name="${name}_depth_frame">
+    <link name="camera_depth_optical_frame">
       <inertial>
         <mass value="0.000001" />
-        <origin xyz="0 0 0" />
+        <origin xyz="0 0 0" rpy="0 0 0" />
         <inertia ixx="0.0001" ixy="0.0" ixz="0.0"
                  iyy="0.0001" iyz="0.0"
@@ -44,13 +130,14 @@
       </inertial>
     </link>
-    <joint name="${name}_depth_optical_joint" type="fixed">
-      <origin xyz="0 0 0" rpy="${-pi/2} 0 ${-pi/2}" />
-      <parent link="${name}_depth_frame" />
-      <child link="${name}_depth_optical_frame" />
+    <!-- camera_color_optical_frame -->
+    <joint name="${name}_rgb_joint" type="fixed">
+      <origin xyz="0.05 0 0.268" rpy="0 0 0" />
+      <parent link="realsense_frame" />
+      <child link="camera_color_optical_frame" />
     </joint>
-    <link name="${name}_depth_optical_frame">
+    <link name="camera_color_optical_frame">
       <inertial>
         <mass value="0.000001" />
-        <origin xyz="0 0 0" />
+        <origin xyz="0 0 0" rpy="0 0 0"/>
         <inertia ixx="0.0001" ixy="0.0" ixz="0.0"
                  iyy="0.0001" iyz="0.0"
@@ -58,32 +145,4 @@
       </inertial>
     </link>
-    <joint name="${name}_rgb_joint" type="fixed">
-      <origin xyz="0.05 0 0.268" rpy="0 0 0" />
-      <parent link="${name}_link" />
-      <child link="${name}_rgb_frame" />
-    </joint>
-    <link name="${name}_rgb_frame">
-      <inertial>
-        <mass value="0.000001" />
-        <origin xyz="0 0 0" />
-        <inertia ixx="0.0001" ixy="0.0" ixz="0.0"
-                 iyy="0.0001" iyz="0.0"
-                 izz="0.0001" />
-      </inertial>
-    </link>
-    <joint name="${name}_rgb_optical_joint" type="fixed">
-      <origin xyz="0 0 0" rpy="${-pi/2} 0 ${-pi/2}" />
-      <parent link="${name}_rgb_frame" />
-      <child link="${name}_rgb_optical_frame" />
-    </joint>
-    <link name="${name}_rgb_optical_frame">
-      <inertial>
-        <mass value="0.000001" />
-       <origin xyz="0 0 0" />
-       <inertia ixx="0.0001" ixy="0.0" ixz="0.0"
-                iyy="0.0001" iyz="0.0"
-                izz="0.0001" />
-      </inertial>
-    </link>
   </macro>
 </robot>

File: robo_description/urdf/robo_two_arms_realsense.xacro (robot description, xacro)
@@ -31,5 +31,5 @@
   </torso>
   <!-- Attach the camera -->
-  <camera name="head_base" parent="torso" color="yellow">
+  <camera name="head" parent="torso" color="yellow">
     <origin xyz="${camera_offset_x} ${camera_offset_y} ${camera_offset_z}" rpy="0 0 ${pi}" />
   </camera>
