Commit message: Minor update

File: robo_description/urdf/robo (copy).urdf (robot description, URDF)
Before this commit: robot robo_hand, 30 links, 29 joints
Joints:
- joint base_joint: origin xyz=0 0 0 rpy=0 0 0 -> xyz=0.0 0.0 0.0 rpy=0 0 0
- joint head_depth_joint: origin xyz=0 0 0 rpy=0 0 0 -> xyz=0 0 0.268 rpy=0 0 0
- joint head_realsense_frame_joint: origin xyz=0 -0.027 0 rpy=0 0 0 -> xyz=0 -0.027 0 rpy=1.570795 3.14159 0
- joint head_rgb_joint: origin xyz=0.05 0 0 rpy=0 0 0 -> xyz=0.05 0 0.268 rpy=0 0 0

File: robo_description/urdf/robo_base.urdf.xacro (robot description, xacro)
@@ -3,20 +3,20 @@
   <!-- Variables  -->
   <property name="pi" value="3.14159"/>
-  <property name="scale" value="0.001" />
-  <property name="base_offset_x" value="0.0" />
-  <property name="base_offset_y" value="0.0" />
-  <property name="base_offset_z" value="0.0" />
+  <property name="scale" value="0.001"/>
+  <property name="base_offset_x" value="0.0"/>
+  <property name="base_offset_y" value="0.0"/>
+  <property name="base_offset_z" value="0.0"/>
   <!-- The base xacro macro -->
   <macro name="base" params="name color">
     <link name="${name}_link">
       <visual>
-        <origin xyz="0 0 0" rpy="0 0 0" />
+        <origin xyz="0 0 0" rpy="0 0 0"/>
         <geometry>
           <mesh filename="package://robo_description/meshes/base/vis/vis_basewheels_03.STL" scale="${scale} ${scale} ${scale}"/>
         </geometry>
-        <material name="${color}" />
+        <material name="${color}"/>
       </visual>
       <collision>
-        <origin xyz="0 0 0" rpy="0 0 0" />
+        <origin xyz="0 0 0" rpy="0 0 0"/>
         <geometry>
           <mesh filename="package://robo_description/meshes/base/col/col_basewheels_03.STL" scale="${scale} ${scale} ${scale}"/>
@@ -26,15 +26,15 @@
     <link name="base_footprint">
         <visual>
-          <origin xyz="0 0 0" rpy="0 0 0" />
+          <origin xyz="0 0 0" rpy="0 0 0"/>
           <geometry>
-            <box size="0.05 0.05 0.001" />
+            <box size="0.05 0.05 0.001"/>
           </geometry>
-          <material name="TransparentGreen" />
+          <material name="TransparentGreen"/>
         </visual>
     </link>
     <joint name="base_joint" type="fixed">
-      <origin xyz="${base_offset_x} ${base_offset_y} ${base_offset_z}" rpy="0 0 0" />
+      <origin xyz="${base_offset_x} ${base_offset_y} ${base_offset_z}" rpy="0 0 0"/>
       <parent link="base_footprint"/>
-      <child link="base_link" />
+      <child link="base_link"/>
     </joint>
   </macro>

File: robo_description/urdf/robo_camera.urdf.xacro (robot description, xacro)
@@ -3,7 +3,7 @@
   <property name="pi" value="3.14159"/>
   <property name="scale" value="0.001" />
-  <property name="camera_offset_x" value="0.0" />
-  <property name="camera_offset_y" value="0.0" />
-  <property name="camera_offset_z" value="0.0" />
+  <property name="camera_offset_x" value="0.0"/>
+  <property name="camera_offset_y" value="0.0"/>
+  <property name="camera_offset_z" value="0.0"/>
   <macro name="camera" params="parent name color *origin">
     <!-- Telescoping neck joint/link -->
@@ -14,9 +14,9 @@
       <axis xyz="0 0 1" />
       <origin xyz="0 0 0" rpy="0 0 0"/>
-      <limit lower="0" upper="0.19" velocity="0.1" effort="1.0" />
+      <limit lower="0" upper="0.19" velocity="0.1" effort="1.0"/>
     </joint>
     <link name="${name}_tele_link">
       <visual>
-        <origin xyz="0 0 0" rpy="0 0 0" />
+        <origin xyz="0 0 0" rpy="0 0 0"/>
         <geometry>
           <box size="0.01 0.01 0.25"/>
@@ -25,5 +25,5 @@
       </visual>
       <collision>
-        <origin xyz="0 0 0" rpy="0 0 0" />
+        <origin xyz="0 0 0" rpy="0 0 0"/>
         <geometry>
           <box size="0.02 0.02 0.5"/>
@@ -41,5 +41,5 @@
     <link name="${name}_pan_link">
       <visual>
-        <origin rpy="0 0 0" xyz="0 0 0"/>
+        <origin xyz="0 0 0" rpy="0 0 0"/>
         <geometry>
           <box size="0.03 0.03 0.03"/>
@@ -48,5 +48,5 @@
       </visual>
       <collision>
-        <origin rpy="0 0 0" xyz="0 0 0"/>
+        <origin xyz="0 0 0" rpy="0 0 0"/>
         <geometry>
           <box size="0.03 0.03 0.03"/>
@@ -71,5 +71,5 @@
       </visual>
       <collision>
-        <origin rpy="0 0 0" xyz="0 0 0"/>
+        <origin xyz="0 0 0" rpy="0 0 0"/>
         <geometry>
           <box size="0.03 0.03 0.01"/>
@@ -79,5 +79,5 @@
     <!-- Realsense joint/link -->
     <joint name="${name}_realsense_joint" type="fixed">
-      <xacro:insert_block name="origin" />
+      <xacro:insert_block name="origin"/>
       <parent link="${name}_tilt_link"/>
       <child link="realsense_link"/>
@@ -85,12 +85,12 @@
     <link name="realsense_link">
       <visual>
-        <origin xyz="0 -0.025 -0.01" rpy="0 0 0" />
+        <origin xyz="0 -0.025 -0.01" rpy="0 0 0"/>
         <geometry>
           <mesh filename="package://robo_description/meshes/camera/vis/RealSense.STL" scale="${scale} ${scale} ${scale}" />
         </geometry>
-        <material name="${color}" />
+        <material name="${color}"/>
       </visual>
       <collision>
-        <origin xyz="0 0 0" rpy="0 0 0" />
+        <origin xyz="0 0 0" rpy="0 0 0"/>
         <geometry>
           <!--box size="0.1 0.02 0.02"/-->
@@ -101,6 +101,6 @@
     <!-- realsense_frame -->
     <joint name="${name}_realsense_frame_joint" type="fixed">
-      <origin xyz="0 -0.027 0" rpy="${pi/2} ${pi} 0" />
-      <xacro:insert_block name="origin" />
+      <origin xyz="0 -0.027 0" rpy="${pi/2} ${pi} 0"/>
+      <!--xacro:insert_block name="origin"/-->
       <parent link="realsense_link"/>
       <child link="realsense_frame"/>
@@ -108,5 +108,5 @@
     <link name="realsense_frame">
       <visual>
-        <origin xyz="0 0 0" rpy="0 0 0" />
+        <origin xyz="0 0 0" rpy="0 0 0"/>
         <geometry>
           <box size="0.003 0.003 0.0005"/>
@@ -117,30 +117,30 @@
     <!-- camera_depth_optical_frame -->
     <joint name="${name}_depth_joint" type="fixed">
-      <origin xyz="0 0 0.268" rpy="0 0 0" />
-      <parent link="realsense_frame" />
-      <child link="camera_depth_optical_frame" />
+      <origin xyz="0 0 0" rpy="0 0 0"/>
+      <parent link="realsense_frame"/>
+      <child link="camera_depth_optical_frame"/>
     </joint>
     <link name="camera_depth_optical_frame">
       <inertial>
-        <mass value="0.000001" />
-        <origin xyz="0 0 0" rpy="0 0 0" />
+        <mass value="0.000001"/>
+        <origin xyz="0 0 0" rpy="0 0 0"/>
         <inertia ixx="0.0001" ixy="0.0" ixz="0.0"
                  iyy="0.0001" iyz="0.0"
-                 izz="0.0001" />
+                 izz="0.0001"/>
       </inertial>
     </link>
     <!-- camera_color_optical_frame -->
     <joint name="${name}_rgb_joint" type="fixed">
-      <origin xyz="0.05 0 0.268" rpy="0 0 0" />
-      <parent link="realsense_frame" />
-      <child link="camera_color_optical_frame" />
+      <origin xyz="0.05 0 0" rpy="0 0 0"/>
+      <parent link="realsense_frame"/>
+      <child link="camera_color_optical_frame"/>
     </joint>
     <link name="camera_color_optical_frame">
       <inertial>
-        <mass value="0.000001" />
+        <mass value="0.000001"/>
         <origin xyz="0 0 0" rpy="0 0 0"/>
         <inertia ixx="0.0001" ixy="0.0" ixz="0.0"
                  iyy="0.0001" iyz="0.0"
-                 izz="0.0001" />
+                 izz="0.0001"/>
       </inertial>
     </link>
