Commit message: Improved arduino code, tweeked urdf

File: robo_description/urdf/materials.urdf.xacro (robot description, xacro)
@@ -53,5 +53,5 @@
     <color rgba="0.0 0.0 0.8 1.0"/>
   </material>
-  <material name="Green">
+    <material name="Green">
     <color rgba="0.0 0.8 0.0 1.0"/>
   </material>

File: robo_description/urdf/robo_arm.urdf.xacro (robot description, xacro)
@@ -1,20 +1,33 @@
 <?xml version="1.0"?>
 <robot name="arm" xmlns:xacro="http://ros.org/wiki/xacro">
+  <!-- Properties -->
   <property name="shouldera_offset_x" value="0.0" />
   <property name="shouldera_offset_y" value="0.5" />
   <property name="shouldera_offset_z" value="0.0" />
-  <xacro:include filename="$(find rbx2_description)/urdf/pi_robot/dynamixel_arm_hardware.xacro" />
+  <!-- Macro -->
   <macro name="arm" params="side reflect parent color *origin">
-    <!-- arm base joint -->
-    <link name="${side}_arm_base_link" />
+    <!-- Arm base -->
+    <!-- L -->
+    <link name="${side}_arm_base_link"/>
+    <!-- J -->
     <joint name="${side}_arm_base_joint" type="fixed">
-      <xacro:insert_block name="origin" />
-      <parent link="${parent}_link" />
-      <child link="${side}_arm_base_link" />
+      <xacro:insert_block name="origin"/>
+      <parent link="${parent}_link"/>
+      <child link="${side}_arm_base_link"/>
     </joint>
-    <!-- Shoulder_A -->
+    <!-- Arm out -->
+    <!-- J -->
+    <joint name="${side}_arm_out_joint" type="revolute">
+      <axis xyz="0 ${-reflect} 0"/>
+      <origin xyz="0 0 0" rpy="0 0 0"/>
+      <xacro:insert_block name="origin"/>
+      <limit effort="1000.0" lower="0.0" upper="${pi/2}" velocity="0.5"/>
+      <parent link="${side}_arm_base_link"/>
+      <child link="${side}_arm_shouldera_link"/>
+    </joint>
+    <!-- L -->
     <link name="${side}_arm_shouldera_link">
       <visual>
-        <origin rpy="0 0 0" xyz="0 0 0"/>
+        <origin xyz="0 0 0" rpy="0 0 0"/>
         <geometry>
           <mesh filename="package://robo_description/meshes/arm/vis/vis_${side}_shouldera_03.STL" scale="${scale} ${scale} ${scale}"/>
@@ -23,5 +36,5 @@
       </visual>
       <collision>
-        <origin rpy="0 0 0" xyz="0 0 0"/>
+        <origin xyz="0 0 0" rpy="0 0 0"/>
         <geometry>
           <mesh filename="package://robo_description/meshes/arm/col/col_${side}_shouldera_03.STL" scale="${scale} ${scale} ${scale}"/>
@@ -29,12 +42,14 @@
       </collision>
     </link>
-    <joint name="${side}_arm_out_joint" type="revolute">
-      <axis xyz="0 ${-reflect} 0"/>
-      <origin rpy="0 0 0" xyz="0 0 0"/>
-      <limit effort="1000.0" lower="0.0" upper="1.5707963" velocity="0.5"/>
-      <parent link="${side}_arm_base_link"/>
-      <child link="${side}_arm_shouldera_link"/>
+    <!-- Arm forward -->
+    <!-- J -->
+    <joint name="${side}_arm_fwd_joint" type="revolute">
+      <axis xyz="-1 0 0"/>
+      <origin xyz="${0.012 * reflect} 0.005 -0.04" rpy="0 0 0"/>
+      <limit effort="1000.0" lower="${-pi/2}" upper="${pi/2}" velocity="0.5"/>
+      <parent link="${side}_arm_shouldera_link"/>
+      <child link="${side}_arm_shoulderb_link"/>
     </joint>
-    <!-- Shoulder_B -->
+    <!-- L -->
     <link name="${side}_arm_shoulderb_link">
       <visual>
@@ -52,15 +67,17 @@
       </collision>
     </link>
-    <joint name="${side}_arm_fwd_joint" type="revolute">
-      <axis xyz="-1 0 0"/>
-      <origin xyz="${0.012 * reflect} 0.005 -0.04" rpy="0 0 0" />
-      <limit effort="1000.0" lower="0.0" upper="${pi/2}" velocity="0.5"/>
-      <parent link="${side}_arm_shouldera_link"/>
-      <child link="${side}_arm_shoulderb_link"/>
+    <!-- Arm rotate -->
+    <!-- J -->
+    <joint name="${side}_arm_rotate_joint" type="revolute">
+      <axis xyz="0 0 ${reflect}"/>
+      <origin xyz="${0.06 * reflect} 0 -0.059" rpy="0 0 0"/>
+      <limit effort="1000.0" lower="${-pi/2}" upper="${pi/2}" velocity="0.5"/>
+      <parent link="${side}_arm_shoulderb_link"/>
+      <child link="${side}_arm_biceps_link"/>
     </joint>
-    <!-- Biceps -->
+    <!-- L -->
     <link name="${side}_arm_biceps_link">
       <visual>
-        <origin xyz="0 0 0" rpy="0 0 0" />
+        <origin xyz="0 0 0" rpy="0 0 0"/>
         <geometry>
           <mesh filename="package://robo_description/meshes/arm/vis/vis_${side}_biceps_03.STL" scale="${scale} ${scale} ${scale}"/>
@@ -75,12 +92,14 @@
       </collision>
     </link>
-    <joint name="${side}_arm_rotate_joint" type="revolute">
-      <axis xyz="0 0 ${reflect}"/>
-      <origin xyz="${0.06 * reflect} 0 -0.059" rpy="0 0 0"/>
-      <limit effort="1000.0" lower="${-pi/2}" upper="${pi/2}" velocity="0.5"/>
-      <parent link="${side}_arm_shoulderb_link"/>
-      <child link="${side}_arm_biceps_link"/>
+    <!-- Elbow -->
+    <!-- J -->
+    <joint name="${side}_elbow_joint" type="revolute">
+      <axis xyz="-1 0 0"/>
+      <origin xyz="0 0.029 -0.225" rpy="0 0 0"/>
+      <limit effort="1000.0" lower="0.0" upper="${pi/2}" velocity="0.5"/>
+      <parent link="${side}_arm_biceps_link"/>
+      <child link="${side}_arm_forearm_link"/>
     </joint>
-    <!-- Forearm -->
+    <!-- L -->
     <link name="${side}_arm_forearm_link">
       <visual>
@@ -92,5 +111,5 @@
       </visual>
       <collision>
-        <origin xyz="0 0 0" rpy="0 0 0" />
+        <origin xyz="0 0 0" rpy="0 0 0"/>
         <geometry>
           <mesh filename="package://robo_description/meshes/arm/col/col_${side}_forearm_03.STL" scale="${scale} ${scale} ${scale}"/>
@@ -98,12 +117,15 @@
       </collision>
     </link>
-    <joint name="${side}_elbow_joint" type="revolute">
-      <axis xyz="-1 0 0"/>
-      <origin xyz="0 0.029 -0.225" rpy="0 0 0"/>
-      <limit effort="1000.0" lower="0.0" upper="${pi/2}" velocity="0.5"/>
-      <parent link="${side}_arm_biceps_link"/>
-      <child link="${side}_arm_forearm_link"/>
+    <!-- Wrist/Hand -->
+    <!-- J -->
+    <joint name="${side}_wrist_joint" type="revolute">
+      <axis xyz="0 0 ${-reflect}"/>
+      <!--origin rpy="0 0 0" xyz=".009972 .012326 -.288718"/-->
+      <origin xyz="0.008 ${-0.01*reflect} -0.2888" rpy="0 0 0"/>
+      <limit effort="1000.0" lower="0.0" upper="${pi}" velocity="0.5"/>
+      <parent link="${side}_arm_forearm_link"/>
+      <child link="${side}_arm_wrist_link"/>
     </joint>
-    <!-- Wrist/Hand -->
+    <!-- L -->
     <link name="${side}_arm_wrist_link">
       <visual>
@@ -121,12 +143,4 @@
       </collision>
     </link>
-    <joint name="${side}_wrist_joint" type="revolute">
-      <axis xyz="0 0 ${-reflect}"/>
-      <!--origin rpy="0 0 0" xyz=".009972 .012326 -.288718"/-->
-      <origin xyz="0.008 ${-0.01*reflect} -0.2888" rpy="0 0 0"/>
-      <limit effort="1000.0" lower="0.0" upper="${pi}" velocity="0.5"/>
-      <parent link="${side}_arm_forearm_link"/>
-      <child link="${side}_arm_wrist_link"/>
-    </joint>
   </macro>
 </robot>

File: robo_description/urdf/robo_base.urdf.xacro (robot description, xacro)
@@ -1,5 +1,5 @@
 <?xml version="1.0"?>
 <robot name="base" xmlns:xacro="http://ros.org/wiki/xacro">
-  <!-- Variables  -->
+  <!-- Properties  -->
   <property name="pi" value="3.14159"/>
   <property name="scale" value="0.001"/>
@@ -7,21 +7,7 @@
   <property name="base_offset_y" value="0.0"/>
   <property name="base_offset_z" value="0.0"/>
-  <!-- The base xacro macro -->
+  <!-- Macro -->
   <macro name="base" params="name color">
-    <link name="${name}_link">
-      <visual>
-        <origin xyz="0 0 0" rpy="0 0 0"/>
-        <geometry>
-          <mesh filename="package://robo_description/meshes/base/vis/vis_basewheels_03.STL" scale="${scale} ${scale} ${scale}"/>
-        </geometry>
-        <material name="${color}"/>
-      </visual>
-      <collision>
-        <origin xyz="0 0 0" rpy="0 0 0"/>
-        <geometry>
-          <mesh filename="package://robo_description/meshes/base/col/col_basewheels_03.STL" scale="${scale} ${scale} ${scale}"/>
-        </geometry>
-      </collision>
-    </link>
+    <!-- L -->
     <link name="base_footprint">
         <visual>
@@ -33,9 +19,27 @@
         </visual>
     </link>
+    <!-- J -->
     <joint name="base_joint" type="fixed">
+      <!--xacro:insert_block name="origin"/-->
       <origin xyz="${base_offset_x} ${base_offset_y} ${base_offset_z}" rpy="0 0 0"/>
       <parent link="base_footprint"/>
       <child link="base_link"/>
     </joint>
+    <!-- L -->
+    <link name="${name}_link">
+      <visual>
+        <origin xyz="0 0 0" rpy="0 0 ${pi}"/>
+        <geometry>
+          <mesh filename="package://robo_description/meshes/base/vis/vis_basewheels_03.STL" scale="${scale} ${scale} ${scale}"/>
+        </geometry>
+        <material name="${color}"/>
+      </visual>
+      <collision>
+        <origin xyz="0 0 0" rpy="0 0 ${pi}"/>
+        <geometry>
+          <mesh filename="package://robo_description/meshes/base/col/col_basewheels_03.STL" scale="${scale} ${scale} ${scale}"/>
+        </geometry>
+      </collision>
+    </link>
   </macro>
 </robot>

File: robo_description/urdf/robo_camera.urdf.xacro (robot description, xacro)
@@ -1,19 +1,22 @@
 <?xml version="1.0"?>
 <robot name="pan_tilt_head" xmlns:xacro="http://ros.org/wiki/xacro">
+  <!-- Properties -->
   <property name="pi" value="3.14159"/>
-  <property name="scale" value="0.001" />
+  <property name="scale" value="0.001"/>
   <property name="camera_offset_x" value="0.0"/>
   <property name="camera_offset_y" value="0.0"/>
   <property name="camera_offset_z" value="0.0"/>
+  <!-- Macro -->
   <macro name="camera" params="parent name color *origin">
-    <!-- Telescoping neck joint/link -->
+    <!-- Telescoping neck -->
+    <!-- J -->
     <joint name="${parent}_${name}_tele_joint" type="prismatic">
-      <xacro:insert_block name="origin" />
+      <xacro:insert_block name="origin"/>
       <parent link="${parent}_link"/>
       <child link="${name}_tele_link"/>
-      <axis xyz="0 0 1" />
-      <origin xyz="0 0 0" rpy="0 0 0"/>
+      <axis xyz="0 0 1"/>
       <limit lower="0" upper="0.19" velocity="0.1" effort="1.0"/>
     </joint>
+    <!-- L -->
     <link name="${name}_tele_link">
       <visual>
@@ -22,5 +25,5 @@
           <box size="0.01 0.01 0.25"/>
         </geometry>
-        <material name="${color}" />
+        <material name="yellow"/>
       </visual>
       <collision>
@@ -31,17 +34,42 @@
       </collision>
     </link>
-    <!-- Pan joint/link -->
+    <!-- Neck to pan fixed -->
+    <!-- J -->
+    <joint name="${name}_neck_joint" type="fixed">
+      <origin xyz="0 0 0.135" rpy="0 0 0"/>
+      <parent link="${name}_tele_link"/>
+      <child link="${name}_neck_link"/>
+    </joint>
+    <!-- L -->
+    <link name="${name}_neck_link">
+      <visual>
+        <origin xyz="0 0 0" rpy="0 0 0"/>
+        <geometry>
+          <box size="0.01 0.03 0.03"/>
+        </geometry>
+        <material name="green"/>
+      </visual>
+      <collision>
+        <origin xyz="0 0 0" rpy="0 0 0"/>
+        <geometry>
+          <box size="0.01 0.03 0.03"/>
+        </geometry>
+      </collision>
+    </link>
+    <!-- Pan -->
+    <!-- J  -->
     <joint name="${name}_pan_joint" type="revolute">
-      <axis xyz="0 0 1"/>
-      <origin xyz="0 0 0.135" rpy="0 0 0"/>
-      <limit effort="1000.0" lower="${pi/2}" upper="${-pi/2}" velocity="0.5"/>
-      <parent link="${name}_tele_link"/>
+      <axis xyz="0 0 -1"/>
+      <origin xyz="0 0 0.02" rpy="0 0 0"/>
+      <limit effort="1000.0" lower="${-pi/2}" upper="${pi/2}" velocity="0.5"/>
+      <parent link="${name}_neck_link"/>
       <child link="${name}_pan_link"/>
     </joint>
+    <!-- L -->
     <link name="${name}_pan_link">
       <visual>
         <origin xyz="0 0 0" rpy="0 0 0"/>
         <geometry>
-          <box size="0.03 0.03 0.03"/>
+          <box size="0.03 0.03 0.01"/>
         </geometry>
         <material name="blue"/>
@@ -50,9 +78,10 @@
         <origin xyz="0 0 0" rpy="0 0 0"/>
         <geometry>
-          <box size="0.03 0.03 0.03"/>
-        </geometry>
-      </collision>
-    </link>
-    <!-- Tilt joint/link -->
+          <box size="0.03 0.03 0.01"/>
+        </geometry>
+      </collision>
+    </link>
+    <!-- Tilt -->
+    <!-- J -->
     <joint name="${name}_tilt_joint" type="revolute">
       <axis xyz="1 0 0"/>
@@ -62,20 +91,22 @@
       <child link="${name}_tilt_link"/>
     </joint>
+    <!-- L -->
     <link name="${name}_tilt_link">
       <visual>
-        <origin xyz="0 0.012 0" rpy="0 0 0"/>
-        <geometry>
-          <box size="0.03 0.03 0.01"/>
-        </geometry>
-        <material name="green"/>
-      </visual>
-      <collision>
-        <origin xyz="0 0 0" rpy="0 0 0"/>
-        <geometry>
-          <box size="0.03 0.03 0.01"/>
-        </geometry>
-      </collision>
-    </link>
-    <!-- Realsense joint/link -->
+        <origin xyz="0 0.01 0" rpy="0 0 0"/>
+        <geometry>
+          <box size="0.035 0.025 0.01"/>
+        </geometry>
+        <material name="indigo"/>
+      </visual>
+      <collision>
+        <origin xyz="0 0.01 0" rpy="0 0 0"/>
+        <geometry>
+          <box size="0.035 0.025 0.01"/>
+        </geometry>
+      </collision>
+    </link>
+    <!-- Realsense body -->
+    <!-- J -->
     <joint name="${name}_realsense_joint" type="fixed">
       <xacro:insert_block name="origin"/>
@@ -83,27 +114,68 @@
       <child link="realsense_link"/>
     </joint>
+    <!-- L -->
     <link name="realsense_link">
       <visual>
-        <origin xyz="0 -0.025 -0.01" rpy="0 0 0"/>
-        <geometry>
-          <mesh filename="package://robo_description/meshes/camera/vis/RealSense.STL" scale="${scale} ${scale} ${scale}" />
-        </geometry>
-        <material name="${color}"/>
-      </visual>
-      <collision>
-        <origin xyz="0 0 0" rpy="0 0 0"/>
-        <geometry>
-          <!--box size="0.1 0.02 0.02"/-->
-          <mesh filename="package://robo_description/meshes/camera/col/col_camera_03.STL" scale="${scale} ${scale} ${scale}" />
-        </geometry>
-      </collision>
+        <origin xyz="0.01 0.025 -0.01" rpy="0 0 ${pi}"/>
+        <geometry>
+          <mesh filename="package://robo_description/meshes/camera/vis/RealSense.STL" scale="${scale} ${scale} ${scale}"/>
+        </geometry>
+        <material name="realsensecolor"/>
+      </visual>
+      <collision>
+        <origin xyz="0.01 0.025 -0.01" rpy="0 0 ${pi}"/>
+        <geometry>
+          <mesh filename="package://robo_description/meshes/camera/col/col_camera_03.STL" scale="${scale} ${scale} ${scale}"/>
+        </geometry>
+      </collision>
+    </link>
+    <!-- Head tracker point A -->
+    <!-- J -->
+    <joint name="${name}_tracker_A_joint" type="fixed">
+      <!--axis xyz="1 1 1"/-->
+      <!--limit effort="1000.0" lower="${pi}" upper="${pi}" velocity="0.5"/-->
+      <!--origin xyz="0 0 0" rpy="${pi/2} ${pi/2} 0"/-->
+      <origin xyz="0 -0.01 0" rpy="${1.57} ${1.57} ${0}"/>
+      <parent link="realsense_link"/>
+      <child link="head_tracker_A_link"/>
+    </joint>
+    <!-- L -->
+    <link name="head_tracker_A_link">
+      <visual>
+        <origin xyz="0 0 0" rpy="0 0 0"/>
+        <geometry>
+          <box size="0.01 0.01 0.01"/>
+        </geometry>
+        <material name="indigo"/>
+      </visual>
+    </link>
+    <!-- Head tracker point B -->
+    <!-- J2 -->
+    <joint name="${name}_tracker_B_joint" type="fixed">
+      <!--axis xyz="1 1 1"/-->
+      <!--limit effort="1000.0" lower="${pi}" upper="${pi}" velocity="0.5"/-->
+      <!--origin xyz="0 0 0" rpy="${pi/2} ${pi/2} 0"/-->
+      <origin xyz="0 0 0" rpy="${pi/5} ${1.57} ${0}"/>
+      <parent link="head_tracker_A_link"/>
+      <child link="head_tracker_B_link"/>
+    </joint>
+    <!-- L2 -->
+    <link name="head_tracker_B_link">
+      <!--visual>
+        <origin xyz="0 0 0" rpy="0 0 0"/>
+        <geometry>
+          <box size="0.01 0.01 0.01"/>
+        </geometry>
+        <material name="orange"/>
+      </visual-->
     </link>
     <!-- realsense_frame -->
+    <!-- J -->
     <joint name="${name}_realsense_frame_joint" type="fixed">
-      <origin xyz="0 -0.027 0" rpy="${pi/2} ${pi} 0"/>
-      <!--xacro:insert_block name="origin"/-->
+      <origin xyz="0.0588 0.027 0.0037" rpy="${pi/2} ${pi} ${pi}"/>
       <parent link="realsense_link"/>
       <child link="realsense_frame"/>
     </joint>
+    <!-- L -->
     <link name="realsense_frame">
       <visual>
@@ -112,8 +184,9 @@
           <box size="0.003 0.003 0.0005"/>
         </geometry>
-        <material name="blue" />
-      </visual>
-    </link>
-    <!-- camera_depth_optical_frame -->
+        <material name="violet"/>
+      </visual>
+    </link>
+    <!-- camera_depth_frame -->
+    <!-- J -->
     <joint name="${name}_depth_joint" type="fixed">
       <origin xyz="0 0 0" rpy="0 0 0"/>
@@ -121,4 +194,5 @@
       <child link="camera_depth_optical_frame"/>
     </joint>
+    <!-- L -->
     <link name="camera_depth_optical_frame">
       <inertial>
@@ -131,10 +205,19 @@
     </link>
     <!-- camera_color_optical_frame -->
+    <!-- J -->
     <joint name="${name}_rgb_joint" type="fixed">
-      <origin xyz="0.05 0 0" rpy="0 0 0"/>
+      <origin xyz="0 0.0003 0" rpy="0 0 0"/>
       <parent link="realsense_frame"/>
       <child link="camera_color_optical_frame"/>
     </joint>
+    <!-- L -->
     <link name="camera_color_optical_frame">
+      <visual>
+        <origin xyz="0 0 0" rpy="0 0 0"/>
+        <geometry>
+          <box size="0.003 0.003 0.001"/>
+        </geometry>
+        <material name="violet"/>
+      </visual>
       <inertial>
         <mass value="0.000001"/>

File: robo_description/urdf/robo_gripper.urdf.xacro (robot description, xacro)
@@ -1,25 +1,38 @@
 <?xml version="1.0"?>
 <robot name="gripper" xmlns:xacro="http://ros.org/wiki/xacro">
+  <!-- Properties -->
   <property name="pi" value="3.14159"/>
   <property name="scale" value="0.001"/>
+  <!-- Macro -->
   <macro name="gripper" params="side reflect parent color *origin">
     <!-- gripper base joint -->
-    <link name="${side}_gripper_base_link" />
+    <!-- L -->
+    <link name="${side}_gripper_base_link"/>
+    <!-- J -->
     <joint name="${side}_gripper_base_joint" type="fixed">
-      <xacro:insert_block name="origin" />
-      <parent link="${parent}_link" />
-      <child link="${side}_gripper_base_link" />
+      <xacro:insert_block name="origin"/>
+      <parent link="${parent}_link"/>
+      <child link="${side}_gripper_base_link"/>
     </joint>
     <!-- Index -->
+    <!-- J -->
+    <joint name="${side}_gripper_index_joint" type="revolute">
+      <origin xyz="${reflect * 0.034} 0 -0.119" rpy="0 0 0"/>
+      <axis xyz="-1 0 0"/>
+      <limit effort="1.0" velocity="3.14" lower="0.0" upper="${pi/2}"/>
+      <parent link="${side}_gripper_base_link"/>
+      <child link="${side}_gripper_index_link"/>
+    </joint>
+    <!-- L -->
     <link name="${side}_gripper_index_link">
       <inertial>
-        <mass value="0.00001" />
-        <origin xyz="0 0 0" />
+        <mass value="0.00001"/>
+        <origin xyz="0 0 0"/>
         <inertia ixx="1.0" ixy="0.0" ixz="0.0"
                  iyy="1.0" iyz="0.0"
-                 izz="1.0" />
+                 izz="1.0"/>
       </inertial>
       <visual>
-        <origin xyz="0 0 0" rpy="0 0 0" />
+        <origin xyz="0 0 0" rpy="0 0 0"/>
         <geometry>
           <mesh filename="package://robo_description/meshes/arm/vis/vis_${side}_index_03.STL" scale="${scale} ${scale} ${scale}"/>
@@ -28,5 +41,5 @@
       </visual>
       <collision>
-        <origin xyz="0 0 0" rpy="0 0 0" />
+        <origin xyz="0 0 0" rpy="0 0 0"/>
         <geometry>
           <mesh filename="package://robo_description/meshes/arm/col/col_${side}_index_03.STL" scale="${scale} ${scale} ${scale}"/>
@@ -34,22 +47,24 @@
       </collision>
     </link>
-    <joint name="${side}_gripper_index_joint" type="revolute">
-      <origin xyz="${reflect * 0.034} 0 -0.119" rpy="0 0 0"/>
-      <axis xyz="-1 0 0"/>
-      <limit effort="1.0" velocity="3.14" lower="0.0" upper="${pi/2}" />
+    <!-- Thumb -->
+    <!-- J -->
+    <joint name="${side}_gripper_thumb_joint" type="revolute">
+      <origin xyz="${reflect * 0.06} 0 -0.0685" rpy="0 0 0"/>
+      <axis xyz="0 0 ${-reflect}"/>
+      <limit effort="1.0" velocity="3.14" lower="0.0" upper="${pi/2}"/>
       <parent link="${side}_gripper_base_link"/>
-      <child link="${side}_gripper_index_link" />
+      <child link="${side}_gripper_thumb_link"/>
     </joint>
-    <!-- Thumb -->
+    <!-- L -->
     <link name="${side}_gripper_thumb_link">
       <inertial>
-        <mass value="0.00001" />
-        <origin xyz="0 0 0" />
+        <mass value="0.00001"/>
+        <origin xyz="0 0 0"/>
         <inertia ixx="1.0" ixy="0.0" ixz="0.0"
                  iyy="1.0" iyz="0.0"
-                 izz="1.0" />
+                 izz="1.0"/>
       </inertial>
       <visual>
-        <origin xyz="0 0 0" rpy="0 0 0" />
+        <origin xyz="0 0 0" rpy="0 0 0"/>
         <geometry>
           <mesh filename="package://robo_description/meshes/arm/vis/vis_${side}_thumb_03.STL" scale="${scale} ${scale} ${scale}"/>
@@ -58,5 +73,5 @@
       </visual>
       <collision>
-        <origin xyz="0 0 0" rpy="0 0 0" />
+        <origin xyz="0 0 0" rpy="0 0 0"/>
         <geometry>
           <mesh filename="package://robo_description/meshes/arm/col/col_${side}_thumb_03.STL" scale="${scale} ${scale} ${scale}"/>
@@ -64,12 +79,12 @@
       </collision>
     </link>
-    <joint name="${side}_gripper_thumb_joint" type="revolute">
-      <origin xyz="${reflect * 0.06} 0 -0.0685" rpy="0 0 0"/>
-      <axis xyz="0 0 ${-reflect}"/>
-      <limit effort="1.0" velocity="3.14" lower="0.0" upper="${pi/2}" />
+    <!-- Fake gripper link and joint for grasp planning -->
+    <!-- J -->
+    <joint name="${side}_gripper_joint" type="fixed">
+      <origin xyz="0 -0.03 -0.09" rpy="${-pi/2} 0 0"/>
       <parent link="${side}_gripper_base_link"/>
-      <child link="${side}_gripper_thumb_link" />
+      <child link="${side}_gripper_link"/>
     </joint>
-    <!-- Fake gripper link and joint for grasp planning -->
+    <!-- L -->
     <link name="${side}_gripper_link">
       <visual>
@@ -86,9 +101,4 @@
       </collision>
     </link>
-    <joint name="${side}_gripper_joint" type="fixed">
-      <origin xyz="0 -0.03 -0.09" rpy="${-pi/2} 0 0"/>
-      <parent link="${side}_gripper_base_link"/>
-      <child link="${side}_gripper_link"/>
-    </joint>
    </macro>
 </robot>
