Commit message: Improved arduino code, tweeked urdf

File: robo_description/urdf/robo_torso.urdf.xacro (robot description, xacro)
@@ -1,31 +1,34 @@
 <?xml version="1.0"?>
 <robot name="torso" xmlns:xacro="http://ros.org/wiki/xacro">
-  <!-- Define a number of dimensions using properties -->
-  <property name="torso_size_x" value="0.0" />
-  <property name="torso_size_y" value="0.0" />
-  <property name="torso_size_z" value="0.0" />
-  <property name="scale" value="0.001" />
-  <!-- Define the torso -->
+  <!-- Properties -->
+  <property name="torso_size_x" value="0.0"/>
+  <property name="torso_size_y" value="0.0"/>
+  <property name="torso_size_z" value="0.0"/>
+  <property name="scale" value="0.001"/>
+  <!-- Macro -->
   <macro name="torso" params="parent name color *origin">
+    <!-- J -->
     <joint name="${parent}_${name}_joint" type="fixed">
-      <xacro:insert_block name="origin" />
+      <xacro:insert_block name="origin"/>
+      <origin xyz="0 0 0" rpy="0 0 0"/>
       <parent link="${parent}_link"/>
       <child link="${name}_link"/>
     </joint>
+    <!-- L -->
     <link name="${name}_link">
       <visual>
-        <origin xyz="0 0 0" rpy="0 0 0" />
+        <origin xyz="0 0 0" rpy="0 0 ${pi}"/>
         <geometry>
-           <mesh filename="package://robo_description/meshes/torso/vis/vis_torso_03.STL" scale="${scale} ${scale} ${scale}" />
+           <mesh filename="package://robo_description/meshes/torso/vis/vis_torso_03.STL" scale="${scale} ${scale} ${scale}"/>
         </geometry>
-        <material name="${color}" />
+        <material name="${color}"/>
       </visual>
       <collision>
-        <origin xyz="0 0 0" rpy="0 0 0" />
+        <origin xyz="0 0 0" rpy="0 0 0"/>
         <geometry>
-          <mesh filename="package://robo_description/meshes/torso/col/col_torso_03.STL" scale="${scale} ${scale} ${scale}" />
+          <mesh filename="package://robo_description/meshes/torso/col/col_torso_03.STL" scale="${scale} ${scale} ${scale}"/>
         </geometry>
       </collision>
-    </link>
+    </link>1`+
   </macro>
 </robot>

File: robo_description/urdf/robo_two_arms_camera.xacro (robot description, xacro)
@@ -1,52 +1,51 @@
 <?xml version="1.0"?>
 <robot name="robo_hand" xmlns:xacro="http://ros.org/wiki/xacro">
-  <!-- Define a number of dimensions using properties -->
+  <!-- Properties -->
   <property name="pi" value="3.14159"/>
-  <property name="torso_offset_x" value="0.0" />
-  <property name="torso_offset_y" value="-0.026" />
-  <property name="torso_offset_z" value="1.255" />
-  <property name="torso_width" value="0.0" />
-  <property name="camera_offset_x" value="0.0" />
-  <property name="camera_offset_y" value="0.0" />
-  <property name="camera_offset_z" value="0.0" />
-  <property name="arm_offset_x" value="-0.143" />
-  <property name="arm_offset_y" value="0.0055" />
-  <property name="arm_offset_z" value="0.047" />
-  <!--property name="arm_offset_x" value="-0.143" /-->
-  <!--property name="arm_offset_y" value="-0.032" /-->
-  <!--property name="arm_offset_z" value="1.302" /-->
-  <!-- Include all component files -->
-  <xacro:include filename="$(find robo_description)/urdf/materials.urdf.xacro" />
-  <xacro:include filename="$(find robo_description)/urdf/robo_base.urdf.xacro" />
-  <xacro:include filename="$(find robo_description)/urdf/robo_torso.urdf.xacro" />
-  <xacro:include filename="$(find robo_description)/urdf/robo_camera.urdf.xacro" />
-  <xacro:include filename="$(find robo_description)/urdf/robo_arm.urdf.xacro" />
-  <xacro:include filename="$(find robo_description)/urdf/robo_gripper.urdf.xacro" />
-  <!-- Now we can start using the macros included above to define the actual robot -->
-  <!-- Add the base and wheels -->
-  <base name="base" color="orange"/>
-  <!-- Attach the torso -->
+  <property name="torso_offset_x" value="0.0"/>
+  <property name="torso_offset_y" value="-0.026"/>
+  <property name="torso_offset_z" value="1.255"/>
+  <property name="torso_width" value="0.0"/>
+  <property name="camera_offset_x" value="0.0"/>
+  <property name="camera_offset_y" value="0.0"/>
+  <property name="camera_offset_z" value="0.0"/>
+  <property name="arm_offset_x" value="-0.143"/>
+  <property name="arm_offset_y" value="0.0055"/>
+  <property name="arm_offset_z" value="0.047"/>
+  <!-- Include files -->
+  <xacro:include filename="$(find robo_description)/urdf/materials.urdf.xacro"/>
+  <xacro:include filename="$(find robo_description)/urdf/robo_base.urdf.xacro"/>
+  <xacro:include filename="$(find robo_description)/urdf/robo_torso.urdf.xacro"/>
+  <xacro:include filename="$(find robo_description)/urdf/robo_camera.urdf.xacro"/>
+  <xacro:include filename="$(find robo_description)/urdf/robo_arm.urdf.xacro"/>
+  <xacro:include filename="$(find robo_description)/urdf/robo_gripper.urdf.xacro"/>
+  <!-- Components -->
+  <!-- Base -->
+  <base name="base" color="orange">
+    <origin xyz="0 0 0" rpy="0 0 0"/>
+  </base>
+  <!-- Torso -->
   <torso name="torso" parent="base" color="red">
-     <origin xyz="${torso_offset_x} ${torso_offset_y} ${torso_offset_z}" rpy="0 0 0" />
+     <origin xyz="${torso_offset_x} ${torso_offset_y} ${torso_offset_z}" rpy="0 0 ${pi}"/>
   </torso>
-  <!-- Attach the camera -->
+  <!-- Head/camera -->
   <camera name="head_base" parent="torso" color="yellow">
-    <origin xyz="${camera_offset_x} ${camera_offset_y} ${camera_offset_z}" rpy="0 0 ${pi}" />
+    <origin xyz="${camera_offset_x} ${camera_offset_y} ${camera_offset_z}" rpy="0 0 0"/>
   </camera>
-  <!-- Attach the right arm -->
+  <!-- Right arm -->
   <arm side="right" reflect="-1" parent="torso" color="green">
-    <origin xyz="${arm_offset_x} ${arm_offset_y} ${arm_offset_z}" rpy="0 0 0" />
+    <origin xyz="${arm_offset_x} ${arm_offset_y} ${arm_offset_z}" rpy="0 0 0"/>
   </arm>
-  <!-- Attach the right gripper -->
+  <!-- Right gripper -->
   <gripper side="right" reflect="-1" parent="right_arm_wrist" color="blue">
-    <origin xyz="0 0 0" rpy="0 0 0" />
+    <origin xyz="0 0 0" rpy="0 0 0"/>
   </gripper>
-  <!-- Attach the left arm -->
+  <!-- Left arm -->
   <arm side="left" reflect="1" parent="torso" color="blue">
-    <origin xyz="${-arm_offset_x} ${arm_offset_y} ${arm_offset_z}" rpy="0 0 0" />
+    <origin xyz="${-arm_offset_x} ${arm_offset_y} ${arm_offset_z}" rpy="0 0 0"/>
   </arm>
-  <!-- Attach the left gripper -->
+  <!-- Left gripper -->
   <gripper side="left" reflect="1" parent="left_arm_wrist" color="blue">
-    <origin xyz="0 0 0" rpy="0 0 0" />
+    <origin xyz="0 0 0" rpy="0 0 0"/>
   </gripper>
 </robot>

File: robo_description/urdf/robo_two_arms_realsense.xacro (robot description, xacro)
@@ -1,8 +1,8 @@
 <?xml version="1.0"?>
 <robot name="robo_hand" xmlns:xacro="http://ros.org/wiki/xacro">
-  <!-- Define a number of dimensions using properties -->
+  <!-- Properties -->
   <property name="pi" value="3.14159"/>
   <property name="torso_offset_x" value="0.0" />
-  <property name="torso_offset_y" value="-0.026" />
+  <property name="torso_offset_y" value="-0.02" />
   <property name="torso_offset_z" value="1.255" />
   <property name="torso_width" value="0.0" />
@@ -10,11 +10,8 @@
   <property name="camera_offset_y" value="0.0" />
   <property name="camera_offset_z" value="0.0" />
-  <property name="arm_offset_x" value="-0.143" />
+  <property name="arm_offset_x" value="0.143" />
   <property name="arm_offset_y" value="0.0055" />
   <property name="arm_offset_z" value="0.047" />
-  <!--property name="arm_offset_x" value="-0.143" /-->
-  <!--property name="arm_offset_y" value="-0.032" /-->
-  <!--property name="arm_offset_z" value="1.302" /-->
-  <!-- Include all component files -->
+  <!-- Include files -->
   <xacro:include filename="$(find robo_description)/urdf/materials.urdf.xacro" />
   <xacro:include filename="$(find robo_description)/urdf/robo_base.urdf.xacro" />
@@ -23,28 +20,28 @@
   <xacro:include filename="$(find robo_description)/urdf/robo_arm.urdf.xacro" />
   <xacro:include filename="$(find robo_description)/urdf/robo_gripper.urdf.xacro" />
-  <!-- Now we can start using the macros included above to define the actual robot -->
-  <!-- Add the base and wheels -->
+  <!-- Components -->
+  <!-- Base -->
   <base name="base" color="orange"/>
-  <!-- Attach the torso -->
+  <!-- Torso -->
   <torso name="torso" parent="base" color="red">
      <origin xyz="${torso_offset_x} ${torso_offset_y} ${torso_offset_z}" rpy="0 0 0" />
   </torso>
-  <!-- Attach the camera -->
+  <!-- Head/camera -->
   <camera name="head" parent="torso" color="yellow">
-    <origin xyz="${camera_offset_x} ${camera_offset_y} ${camera_offset_z}" rpy="0 0 ${pi}" />
+    <origin xyz="${camera_offset_x} ${camera_offset_y} ${camera_offset_z}" rpy="0 0 0" />
   </camera>
-  <!-- Attach the right arm -->
+  <!-- Right arm -->
   <arm side="right" reflect="-1" parent="torso" color="green">
-    <origin xyz="${arm_offset_x} ${arm_offset_y} ${arm_offset_z}" rpy="0 0 0" />
+    <origin xyz="${arm_offset_x} ${arm_offset_y} ${arm_offset_z}" rpy="0 0 ${pi}" />
   </arm>
-  <!-- Attach the right gripper -->
+  <!-- Right gripper -->
   <gripper side="right" reflect="-1" parent="right_arm_wrist" color="blue">
     <origin xyz="0 0 0" rpy="0 0 0" />
   </gripper>
-  <!-- Attach the left arm -->
+  <!-- Left arm -->
   <arm side="left" reflect="1" parent="torso" color="blue">
-    <origin xyz="${-arm_offset_x} ${arm_offset_y} ${arm_offset_z}" rpy="0 0 0" />
+    <origin xyz="${-arm_offset_x} ${arm_offset_y} ${arm_offset_z}" rpy="0 0 ${pi}" />
   </arm>
-  <!-- Attach the left gripper -->
+  <!-- Left gripper -->
   <gripper side="left" reflect="1" parent="left_arm_wrist" color="blue">
     <origin xyz="0 0 0" rpy="0 0 0" />
