Commit message: Update robot model with new head collision. Redo Moveit! setup assistant

File: robo_description/urdf/robo.urdf (robot description, URDF)
Before this commit: robot robo_hand, 30 links, 29 joints
Links:
- added link head_col_link; collision box size=0.15 0.15 0.25; visual box size=0.01 0.01 0.01
- added link head_neck_link; visual box size=0.01 0.03 0.03
- added link head_tracker_A_link; visual box size=0.01 0.01 0.01
- added link head_tracker_B_link
- link camera_color_optical_frame: geometry visual box size=0.003 0.003 0.001
- link head_pan_link: geometry visual box size=0.03 0.03 0.01
- link head_tele_link: geometry visual box size=0.01 0.01 0.25
- link head_tilt_link: geometry visual box size=0.035 0.025 0.01
- link realsense_link: geometry visual mesh filename=package://robo_description/meshes/camera/vis/RealSense.STL scale=0.001 0.001 0.001
Joints:
- added joint head_col_joint: type fixed, parent torso_link, child head_col_link, origin xyz=0 0 0.24 rpy=0 0 0
- added joint head_neck_joint: type fixed, parent head_tele_link, child head_neck_link, origin xyz=0 0 0.135 rpy=0 0 0
- added joint head_tracker_A_joint: type fixed, parent realsense_link, child head_tracker_A_link, origin xyz=0 -0.01 0 rpy=1.57 1.57 0.0
- added joint head_tracker_B_joint: type fixed, parent head_tracker_A_link, child head_tracker_B_link, origin xyz=0 0 0 rpy=0.628318 1.57 0.0
- joint base_joint: origin xyz=0 0 0 rpy=0 0 0 -> xyz=0.0 0.0 0.0 rpy=0 0 0
- joint base_torso_joint: origin xyz=0.0 -0.026 1.255 rpy=0 0 0 -> xyz=0.0 -0.02 1.255 rpy=0 0 0
- joint head_pan_joint: axis 0 0 1 -> 0 0 -1; limit lower=1.570795 upper=-1.570795 effort=1000.0 velocity=0.5 -> lower=-1.570795 upper=1.570795 effort=1000.0 velocity=0.5; origin xyz=0 0 0.135 rpy=0 0 0 -> xyz=0 0 0.02 rpy=0 0 0; parent head_tele_link -> head_neck_link
- joint head_realsense_frame_joint: origin xyz=0 -0.027 0 rpy=0 0 0 -> xyz=0.0588 0.027 0.0037 rpy=1.570795 3.14159 3.14159
- joint head_realsense_joint: origin xyz=0.0 0.0 0.0 rpy=0 0 3.14159 -> xyz=0.0 0.0 0.0 rpy=0 0 0
- joint head_rgb_joint: origin xyz=0.05 0 0 rpy=0 0 0 -> xyz=0 0.0003 0 rpy=0 0 0
- joint left_arm_base_joint: origin xyz=0.143 0.0055 0.047 rpy=0 0 0 -> xyz=-0.143 0.0055 0.047 rpy=0 0 3.14159
- joint left_arm_fwd_joint: limit lower=0.0 upper=1.570795 effort=1000.0 velocity=0.5 -> lower=-1.570795 upper=1.570795 effort=1000.0 velocity=0.5
- joint left_arm_out_joint: limit lower=0.0 upper=1.5707963 effort=1000.0 velocity=0.5 -> lower=0.0 upper=1.570795 effort=1000.0 velocity=0.5
- joint right_arm_base_joint: origin xyz=-0.143 0.0055 0.047 rpy=0 0 0 -> xyz=0.143 0.0055 0.047 rpy=0 0 3.14159
- joint right_arm_fwd_joint: limit lower=0.0 upper=1.570795 effort=1000.0 velocity=0.5 -> lower=-1.570795 upper=1.570795 effort=1000.0 velocity=0.5
- joint right_arm_out_joint: limit lower=0.0 upper=1.5707963 effort=1000.0 velocity=0.5 -> lower=0.0 upper=1.570795 effort=1000.0 velocity=0.5
- joint torso_head_tele_joint: origin xyz=0.0 0.0 0.0 rpy=0 0 3.14159 -> xyz=0.0 0.0 0.0 rpy=0 0 0

File: robo_description/urdf/robo_camera.urdf.xacro (robot description, xacro)
@@ -27,10 +27,10 @@
         <material name="yellow"/>
       </visual>
-      <collision>
+      <!--collision>
         <origin xyz="0 0 0" rpy="0 0 0"/>
         <geometry>
           <box size="0.02 0.02 0.5"/>
         </geometry>
-      </collision>
+      </collision!-->
     </link>
     <!-- Neck to pan fixed -->
@@ -42,4 +42,5 @@
     </joint>
     <!-- L -->
+    <!-- This contains the head collision box -->
     <link name="${name}_neck_link">
       <visual>
@@ -50,10 +51,10 @@
         <material name="green"/>
       </visual>
-      <collision>
-        <origin xyz="0 0 0" rpy="0 0 0"/>
-        <geometry>
-          <box size="0.01 0.03 0.03"/>
-        </geometry>
-      </collision>
+      <!--collision>
+        <origin xyz="0 0 0.1" rpy="0 0 0"/>
+        <geometry>
+          <box size="0.2 0.2 0.2"/>
+        </geometry>
+      </collision!-->
     </link>
     <!-- Pan -->
@@ -75,10 +76,10 @@
         <material name="blue"/>
       </visual>
-      <collision>
+      <!--collision>
         <origin xyz="0 0 0" rpy="0 0 0"/>
         <geometry>
           <box size="0.03 0.03 0.01"/>
         </geometry>
-      </collision>
+      </collision!-->
     </link>
     <!-- Tilt -->
@@ -100,10 +101,10 @@
         <material name="indigo"/>
       </visual>
-      <collision>
+      <!--collision>
         <origin xyz="0 0.01 0" rpy="0 0 0"/>
         <geometry>
           <box size="0.035 0.025 0.01"/>
         </geometry>
-      </collision>
+      </collision!-->
     </link>
     <!-- Realsense body -->
@@ -123,10 +124,10 @@
         <material name="realsensecolor"/>
       </visual>
-      <collision>
+      <!--collision>
         <origin xyz="0.01 0.025 -0.01" rpy="0 0 ${pi}"/>
         <geometry>
           <mesh filename="package://robo_description/meshes/camera/col/col_camera_03.STL" scale="${scale} ${scale} ${scale}"/>
         </geometry>
-      </collision>
+      </collision!-->
     </link>
     <!-- Head tracker point A -->

File: robo_description/urdf/robo_torso.urdf.xacro (robot description, xacro)
@@ -30,5 +30,26 @@
         </geometry>
       </collision>
-    </link>1`+
+    </link>
+    <!-- J -->
+    <joint name="head_col_joint" type="fixed">
+      <origin xyz="0 0 0.24" rpy="0 0 0"/>
+      <parent link="${name}_link"/>
+      <child link="head_col_link"/>
+    </joint>
+    <!-- L -->
+    <link name="head_col_link">
+      <visual>
+        <origin xyz="0 0 0" rpy="0 0 0"/>
+        <geometry>
+          <box size="0.01 0.01 0.01"/>
+        </geometry>
+      </visual>
+      <collision>
+        <origin xyz="0 0 0" rpy="0 0 0"/>
+        <geometry>
+          <box size="0.15 0.15 0.25"/>
+        </geometry>
+      </collision>
+    </link>
   </macro>
 </robot>

Commit message: Improved translate node, added sep topics for each limb. Improved Arduino node. Developed trajectory.demo.py

File: robo_description/urdf/robo.urdf (robot description, URDF)
Before this commit: robot robo_hand, 34 links, 33 joints
Links:
- link head_col_link: geometry collision box size=0.15 0.15 0.25

File: robo_description/urdf/robo_arm.urdf.xacro (robot description, xacro)
@@ -33,5 +33,5 @@
           <mesh filename="package://robo_description/meshes/arm/vis/vis_${side}_shouldera_03.STL" scale="${scale} ${scale} ${scale}"/>
         </geometry>
-        <material name="orange"/>
+        <material name="${color}"/>
       </visual>
       <collision>
@@ -58,5 +58,5 @@
           <mesh filename="package://robo_description/meshes/arm/vis/vis_${side}_shoulderb_03.STL" scale="${scale} ${scale} ${scale}"/>
         </geometry>
-        <material name="yellow"/>
+        <material name="${color}"/>
       </visual>
       <collision>
@@ -83,5 +83,5 @@
           <mesh filename="package://robo_description/meshes/arm/vis/vis_${side}_biceps_03.STL" scale="${scale} ${scale} ${scale}"/>
         </geometry>
-        <material name="green"/>
+        <material name="${color}"/>
       </visual>
       <collision>
@@ -108,5 +108,5 @@
           <mesh filename="package://robo_description/meshes/arm/vis/vis_${side}_forearm_03.STL" scale="${scale} ${scale} ${scale}"/>
         </geometry>
-        <material name="blue"/>
+        <material name="${color}"/>
       </visual>
       <collision>
@@ -134,5 +134,5 @@
           <mesh filename="package://robo_description/meshes/arm/vis/vis_${side}_hand_03.STL" scale="${scale} ${scale} ${scale}"/>
         </geometry>
-        <material name="indigo"/>
+        <material name="${color}"/>
       </visual>
       <collision>

File: robo_description/urdf/robo_camera.urdf.xacro (robot description, xacro)
@@ -25,5 +25,5 @@
           <box size="0.01 0.01 0.25"/>
         </geometry>
-        <material name="yellow"/>
+        <material name="${color}"/>
       </visual>
       <!--collision>
@@ -49,5 +49,5 @@
           <box size="0.01 0.03 0.03"/>
         </geometry>
-        <material name="green"/>
+        <material name="${color}"/>
       </visual>
       <!--collision>
@@ -74,5 +74,5 @@
           <box size="0.03 0.03 0.01"/>
         </geometry>
-        <material name="blue"/>
+        <material name="${color}"/>
       </visual>
       <!--collision>
@@ -99,5 +99,5 @@
           <box size="0.035 0.025 0.01"/>
         </geometry>
-        <material name="indigo"/>
+        <material name="${color}"/>
       </visual>
       <!--collision>
@@ -120,5 +120,5 @@
         <origin xyz="0.01 0.025 -0.01" rpy="0 0 ${pi}"/>
         <geometry>
-          <mesh filename="package://robo_description/meshes/camera/vis/RealSense.STL" scale="${scale} ${scale} ${scale}"/>
+          <mesh filename="package://robo_description/meshes/camera/vis/RealSense.STL" scale="${scale} ${scale} ${scale}"/>z
         </geometry>
         <material name="realsensecolor"/>
@@ -148,5 +148,5 @@
           <box size="0.01 0.01 0.01"/>
         </geometry>
-        <material name="indigo"/>
+        <material name="${color}"/>
       </visual>
     </link>
@@ -185,5 +185,5 @@
           <box size="0.003 0.003 0.0005"/>
         </geometry>
-        <material name="violet"/>
+        <material name="${color}"/>
       </visual>
     </link>
@@ -219,5 +219,5 @@
           <box size="0.003 0.003 0.001"/>
         </geometry>
-        <material name="violet"/>
+        <material name="${color}"/>
       </visual>
       <inertial>

File: robo_description/urdf/robo_gripper.urdf.xacro (robot description, xacro)
@@ -38,5 +38,5 @@
           <mesh filename="package://robo_description/meshes/arm/vis/vis_${side}_index_03.STL" scale="${scale} ${scale} ${scale}"/>
         </geometry>
-        <material name="violet"/>
+        <material name="${color}"/>
       </visual>
       <collision>
@@ -70,5 +70,5 @@
           <mesh filename="package://robo_description/meshes/arm/vis/vis_${side}_thumb_03.STL" scale="${scale} ${scale} ${scale}"/>
         </geometry>
-        <material name="violet"/>
+        <material name="${color}"/>
       </visual>
       <collision>

File: robo_description/urdf/robo_torso.urdf.xacro (robot description, xacro)
@@ -39,10 +39,11 @@
     <!-- L -->
     <link name="head_col_link">
-      <visual>
+      <!--visual>
         <origin xyz="0 0 0" rpy="0 0 0"/>
         <geometry>
           <box size="0.01 0.01 0.01"/>
         </geometry>
-      </visual>
+        <material name="TransparentGreen"/>
+      </visual-->
       <collision>
         <origin xyz="0 0 0" rpy="0 0 0"/>

File: robo_description/urdf/robo_two_arms_realsense.xacro (robot description, xacro)
@@ -3,47 +3,47 @@
   <!-- Properties -->
   <property name="pi" value="3.14159"/>
-  <property name="torso_offset_x" value="0.0" />
-  <property name="torso_offset_y" value="-0.02" />
-  <property name="torso_offset_z" value="1.255" />
-  <property name="torso_width" value="0.0" />
-  <property name="camera_offset_x" value="0.0" />
-  <property name="camera_offset_y" value="0.0" />
-  <property name="camera_offset_z" value="0.0" />
-  <property name="arm_offset_x" value="0.143" />
-  <property name="arm_offset_y" value="0.0055" />
-  <property name="arm_offset_z" value="0.047" />
+  <property name="torso_offset_x" value="0.0"/>
+  <property name="torso_offset_y" value="-0.02"/>
+  <property name="torso_offset_z" value="1.255"/>
+  <property name="torso_width" value="0.0"/>
+  <property name="camera_offset_x" value="0.0"/>
+  <property name="camera_offset_y" value="0.0"/>
+  <property name="camera_offset_z" value="0.0"/>
+  <property name="arm_offset_x" value="0.143"/>
+  <property name="arm_offset_y" value="0.0055"/>
+  <property name="arm_offset_z" value="0.047"/>
   <!-- Include files -->
-  <xacro:include filename="$(find robo_description)/urdf/materials.urdf.xacro" />
-  <xacro:include filename="$(find robo_description)/urdf/robo_base.urdf.xacro" />
-  <xacro:include filename="$(find robo_description)/urdf/robo_torso.urdf.xacro" />
-  <xacro:include filename="$(find robo_description)/urdf/robo_camera.urdf.xacro" />
-  <xacro:include filename="$(find robo_description)/urdf/robo_arm.urdf.xacro" />
-  <xacro:include filename="$(find robo_description)/urdf/robo_gripper.urdf.xacro" />
+  <xacro:include filename="$(find robo_description)/urdf/materials.urdf.xacro"/>
+  <xacro:include filename="$(find robo_description)/urdf/robo_base.urdf.xacro"/>
+  <xacro:include filename="$(find robo_description)/urdf/robo_torso.urdf.xacro"/>
+  <xacro:include filename="$(find robo_description)/urdf/robo_camera.urdf.xacro"/>
+  <xacro:include filename="$(find robo_description)/urdf/robo_arm.urdf.xacro"/>
+  <xacro:include filename="$(find robo_description)/urdf/robo_gripper.urdf.xacro"/>
   <!-- Components -->
   <!-- Base -->
-  <base name="base" color="orange"/>
+  <base name="base" color="DarkGrey"/>
   <!-- Torso -->
-  <torso name="torso" parent="base" color="red">
-     <origin xyz="${torso_offset_x} ${torso_offset_y} ${torso_offset_z}" rpy="0 0 0" />
+  <torso name="torso" parent="base" color="Grey">
+     <origin xyz="${torso_offset_x} ${torso_offset_y} ${torso_offset_z}" rpy="0 0 0"/>
   </torso>
   <!-- Head/camera -->
-  <camera name="head" parent="torso" color="yellow">
-    <origin xyz="${camera_offset_x} ${camera_offset_y} ${camera_offset_z}" rpy="0 0 0" />
+  <camera name="head" parent="torso" color="DarkGrey">
+    <origin xyz="${camera_offset_x} ${camera_offset_y} ${camera_offset_z}" rpy="0 0 0"/>
   </camera>
   <!-- Right arm -->
-  <arm side="right" reflect="-1" parent="torso" color="green">
-    <origin xyz="${arm_offset_x} ${arm_offset_y} ${arm_offset_z}" rpy="0 0 ${pi}" />
+  <arm side="right" reflect="-1" parent="torso" color="DarkGrey">
+    <origin xyz="${arm_offset_x} ${arm_offset_y} ${arm_offset_z}" rpy="0 0 ${pi}"/>
   </arm>
   <!-- Right gripper -->
-  <gripper side="right" reflect="-1" parent="right_arm_wrist" color="blue">
-    <origin xyz="0 0 0" rpy="0 0 0" />
+  <gripper side="right" reflect="-1" parent="right_arm_wrist" color="Grey">
+    <origin xyz="0 0 0" rpy="0 0 0"/>
   </gripper>
   <!-- Left arm -->
-  <arm side="left" reflect="1" parent="torso" color="blue">
-    <origin xyz="${-arm_offset_x} ${arm_offset_y} ${arm_offset_z}" rpy="0 0 ${pi}" />
+  <arm side="left" reflect="1" parent="torso" color="DarkGrey">
+    <origin xyz="${-arm_offset_x} ${arm_offset_y} ${arm_offset_z}" rpy="0 0 ${pi}"/>
   </arm>
   <!-- Left gripper -->
-  <gripper side="left" reflect="1" parent="left_arm_wrist" color="blue">
-    <origin xyz="0 0 0" rpy="0 0 0" />
+  <gripper side="left" reflect="1" parent="left_arm_wrist" color="Grey">
+    <origin xyz="0 0 0" rpy="0 0 0"/>
   </gripper>
 </robot>
